Commit message: Add files via upload

File: objects/totem_banane.urdf (robot description, URDF)
Before this commit: robot physics, 4 links, 3 joints
Links:
- link banane_stuff: geometry collision mesh filename=Totem_banane/banane.obj scale=.03 .03 .03; visual mesh filename=Totem_banane/banane.obj scale=.01 .01 .01
