Commit message: Add files via upload

File: objects/totem_pomme.urdf (robot description, URDF)
Before this commit: robot physics, 4 links, 3 joints
Links:
- link pomme_stuff: geometry collision mesh filename=Totem_pomme/pomme.obj scale=.00005 .00005 .00005; visual mesh filename=Totem_pomme/pomme.obj scale=.0003 .0003 .0003

Commit message: Add files via upload

File: objects/totem_pomme.urdf (robot description, URDF)
Before this commit: robot physics, 4 links, 3 joints
Links:
- link pomme_stuff: geometry collision mesh filename=Totem_pomme/apple.obj scale=.01 .01 .01; visual mesh filename=Totem_pomme/apple.obj scale=.01 .01 .01
