Commit message: Update totem_raquette.urdf

File: objects/totem_raquette.urdf (robot description, URDF)
Before this commit: robot physics, 4 links, 3 joints
Links:
- link raquette_stuff: geometry collision mesh filename=Totem_raquette/raquette.obj scale=.008 .008 .008; visual mesh filename=Totem_raquette/raquette.obj scale=.003 .003 .003

Commit message: Add files via upload

File: objects/totem_raquette.urdf (robot description, URDF)
Before this commit: robot physics, 4 links, 3 joints
Links:
- link raquette_stuff: geometry collision mesh filename=Totem_raquette/raquette.obj scale=.003 .003 .003; visual mesh filename=Totem_raquette/raquette.obj scale=.003 .003 .003
