Commit message: Add files via upload

File: objects/totem_avion.urdf (robot description, URDF)
Before this commit: robot physics, 4 links, 3 joints
Links:
- link avion_stuff: geometry collision mesh filename=Totem_avion/avion.obj scale=.00005 .00005 .00005; visual mesh filename=Totem_avion/avion.obj scale=.00008 .00008 .00008

File: objects/totem_banane.urdf (robot description, URDF)
Before this commit: robot physics, 4 links, 3 joints
Links:
- link banane_stuff: geometry collision mesh filename=Totem_banane/banane.obj scale=.02 .02 .02; visual mesh filename=Totem_banane/banane.obj scale=.02 .02 .02

File: objects/totem_pomme.urdf (robot description, URDF)
Before this commit: robot physics, 4 links, 3 joints
Links:
- removed link pomme_stuff
- added link raquette_stuff, mass .001; collision mesh filename=Totem_pomme/raquette.obj scale=.008 .008 .008; visual mesh filename=Totem_pomme/raquette.obj scale=.003 .003 .003
Joints:
- joint jfixed_stuff: child pomme_stuff -> raquette_stuff

Commit message: Add files via upload

File: objects/totem_avion.urdf (robot description, URDF)
Before this commit: robot physics, 4 links, 3 joints
Links:
- link avion_stuff: geometry collision mesh filename=Totem_avion/avion.obj scale=.00008 .00008 .00008; visual mesh filename=Totem_avion/avion.obj scale=.00008 .00008 .00008

File: objects/totem_raquette.urdf (robot description, URDF)
Before this commit: robot physics, 4 links, 3 joints
Links:
- link raquette_stuff: geometry collision mesh filename=Totem_raquette/raquette.obj scale=.008 .008 .008; visual mesh filename=Totem_raquette/raquette.obj scale=.003 .003 .003
