Commit message: Add files via upload

File: objects/totem_incendie.urdf (robot description, URDF)
Before this commit: robot physics, 4 links, 3 joints
Links:
- removed link raquette_stuff
- added link fourchette_stuff, mass .001; collision mesh filename=Totem_incendie/BAI.obj scale=.002 .002 .002; visual mesh filename=Totem_incendie/BAI.obj scale=.002 .002 .002
Joints:
- joint jfixed_stuff: child raquette_stuff -> fourchette_stuff
