Commit message: nouvelle boite2 avec collision

File: objects/boite/box2.urdf (robot description, URDF)
Before this commit: robot box2.urdf, 1 links, 0 joints
Links:
- link baseLink: geometry collision mesh filename=boite/Boite2.obj scale=.03 .03 .03; visual mesh filename=boite/Boite2.obj scale=.03 .03 .03

Commit message: Update box2.urdf

File: objects/boite/box2.urdf (robot description, URDF)
Before this commit: robot box2.urdf, 1 links, 0 joints
Links:
- link baseLink: geometry collision mesh filename=boite/Boite2.obj scale=.03 .03 .03; visual mesh filename=boite/box2.obj scale=.03 .03 .03
