Commit message: nouvelle boite3 avec collision

File: objects/boite/box3.urdf (robot description, URDF)
Before this commit: robot box.urdf, 1 links, 0 joints
Links:
- link baseLink: geometry collision mesh filename=boite/Boite3.obj scale=.02 .02 .02; visual mesh filename=boite/Boite3.obj scale=.03 .03 .03

Commit message: Update box3.urdf

File: objects/boite/box3.urdf (robot description, URDF)
Before this commit: robot box.urdf, 1 links, 0 joints
Links:
- link baseLink: geometry collision mesh filename=boite/Boite3.obj scale=.02 .02 .02; visual mesh filename=boite/osier.obj scale=.03 .03 .03
