Commit message: Add files via upload

File: objects/boite/boite.urdf (robot description, URDF)
Before this commit: robot boite.urdf, 1 links, 0 joints
Links:
- link baseLink: geometry collision mesh filename=boite/box.obj scale=.02 .02 .02; visual mesh filename=boite/box.obj scale=.015 .015 .015

Commit message: nouvelle boite1 avec collisioin

File: objects/boite/boite.urdf (robot description, URDF)
Before this commit: robot box.urdf, 1 links, 0 joints
Links:
- link baseLink: geometry collision mesh filename=boite/Boite1.obj scale=.02 .02 .02; visual mesh filename=boite/Boite1.obj scale=.015 .015 .015

Commit message: Update boite.urdf

File: objects/boite/boite.urdf (robot description, URDF)
Before this commit: robot box.urdf, 1 links, 0 joints
Links:
- link baseLink: geometry collision mesh filename=boite/Boite1.obj scale=.02 .02 .02; visual mesh filename=boite/box.obj scale=.015 .015 .015

Commit message: Add files via upload

File: objects/boite/boite.urdf (robot description, URDF)
Before this commit: robot box.urdf, 1 links, 0 joints
Links:
- link baseLink: geometry collision mesh filename=boite/Boite1.obj scale=.02 .02 .02; visual mesh filename=boite/box.obj scale=.010 .010 .010

File: objects/boite/box2.urdf (robot description, URDF)
Before this commit: robot box2.urdf, 1 links, 0 joints
Links:
- link baseLink: geometry collision mesh filename=boite/Boite2.obj scale=.03 .03 .03; visual mesh filename=boite/box2.obj scale=.02 .02 .02

File: objects/boite/box3.urdf (robot description, URDF)
Before this commit: robot box.urdf, 1 links, 0 joints
Links:
- link baseLink: geometry collision mesh filename=boite/Boite3.obj scale=.02 .02 .02; visual mesh filename=boite/osier.obj scale=.02 .02 .02

Commit message: Add files via upload

File: objects/boite/boite.urdf (robot description, URDF)
Before this commit: robot box.urdf, 1 links, 0 joints
Links:
- link baseLink: geometry collision mesh filename=boite/Boite1.obj scale=.01 .01 .01; visual mesh filename=boite/box.obj scale=.010 .010 .010

File: objects/boite/box2.urdf (robot description, URDF)
Before this commit: robot box2.urdf, 1 links, 0 joints
Links:
- link baseLink: geometry collision mesh filename=boite/Boite2.obj scale=.02 .02 .02; visual mesh filename=boite/box2.obj scale=.02 .02 .02

Commit message: Add files via upload

File: objects/boite/boite.urdf (robot description, URDF)
Before this commit: robot box.urdf, 1 links, 0 joints
Links:
- link baseLink: geometry collision mesh filename=boite/boite1.obj scale=.015 .015 .015; visual mesh filename=boite/box.obj scale=.015 .015 .015

File: objects/boite/box2.urdf (robot description, URDF)
Before this commit: robot box2.urdf, 1 links, 0 joints
Links:
- link baseLink: geometry collision mesh filename=boite/box2.obj scale=.03 .03 .03; visual mesh filename=boite/box2.obj scale=.03 .03 .03

File: objects/boite/box3.urdf (robot description, URDF)
Before this commit: robot box.urdf, 1 links, 0 joints
Links:
- link baseLink: geometry collision mesh filename=boite/osier.obj scale=.03 .03 .03; visual mesh filename=boite/osier.obj scale=.03 .03 .03

Commit message: Add files via upload

File: objects/boite/boite.urdf (robot description, URDF)
Before this commit: robot box.urdf, 1 links, 0 joints
Links:
- link baseLink: geometry collision mesh filename=Boite1.obj scale=.015 .015 .015; visual mesh filename=box.obj scale=.015 .015 .015

File: objects/boite/box2.urdf (robot description, URDF)
Before this commit: robot box2.urdf, 1 links, 0 joints
Links:
- link baseLink: geometry collision mesh filename=Boite2.obj scale=.03 .03 .03; visual mesh filename=box2.obj scale=.03 .03 .03

File: objects/boite/box3.urdf (robot description, URDF)
Before this commit: robot box.urdf, 1 links, 0 joints
Links:
- link baseLink: geometry collision mesh filename=Boite3.obj scale=.03 .03 .03; visual mesh filename=osier.obj scale=.03 .03 .03

Commit message: Add files via upload

File: objects/boite/boite.urdf (robot description, URDF)
Before this commit: robot box.urdf, 1 links, 0 joints
Links:
- link baseLink: geometry collision mesh filename=Boite1.obj scale=.01 .01 .01; visual mesh filename=box.obj scale=.01 .01 .01

File: objects/boite/box2.urdf (robot description, URDF)
Before this commit: robot box2.urdf, 1 links, 0 joints
Links:
- link baseLink: geometry collision mesh filename=Boite2.obj scale=.02 .02 .02; visual mesh filename=box2.obj scale=.02 .02 .02

File: objects/boite/box3.urdf (robot description, URDF)
Before this commit: robot box.urdf, 1 links, 0 joints
Links:
- link baseLink: geometry collision mesh filename=Boite3.obj scale=.02 .02 .02; visual mesh filename=osier.obj scale=.02 .02 .02
